Commit message: Stuck to fix the assmebled urdf

File: install/robot_description/share/robot_description/urdf/gazebo.xacro (robot description, xacro)
@@ -1,3 +1,31 @@
 <?xml version="1.0"?>
 <robot xmlns:xacro="http://www.ros.org/wiki/xacro">
+    <!-- Gazebo Material Overrides -->
+    <gazebo reference="base_link">
+        <material>Gazebo/Grey</material>
+    </gazebo>
+    <gazebo reference="link1">
+        <material>Gazebo/Grey</material>
+    </gazebo>
+    <gazebo reference="link2">
+        <material>Gazebo/Grey</material>
+    </gazebo>
+    <gazebo reference="link3">
+        <material>Gazebo/Grey</material>
+    </gazebo>
+    <gazebo reference="link4">
+        <material>Gazebo/Grey</material>
+    </gazebo>
+    <gazebo reference="link5">
+        <material>Gazebo/Grey</material>
+    </gazebo>
+    <gazebo reference="link6">
+        <material>Gazebo/Grey</material>
+    </gazebo>
+    <!-- Contact Parameters -->
+    <gazebo reference="base_link">
+        <mu1>1.0</mu1>
+        <mu2>1.0</mu2>
+        <selfCollide>false</selfCollide>
+    </gazebo>
 </robot>

File: install/robot_description/share/robot_description/urdf/joints.xacro (robot description, xacro)
@@ -7,9 +7,9 @@
         <parent link="base_link"/>
         <child link="link1"/>
-        <origin xyz="0 0 0.10" rpy="0 0 0"/>
+        <origin xyz="0 0 0.0405" rpy="0 0 0"/>
         <axis xyz="0 0 1"/>
         <limit
-            lower="-2.79"
-            upper="2.79"
+            lower="-3.14159"
+            upper="3.14159"
             effort="100"
             velocity="2.0"/>
@@ -21,7 +21,7 @@
         <parent link="link1"/>
         <child link="link2"/>
-        <origin xyz="0 0 0.15"
-                rpy="-1.5708 0 0"/>
-        <axis xyz="0 0 1"/>
+        <origin xyz="0.020 -0.0396 0.1045"
+                rpy="0 0 0"/>
+        <axis xyz="0 1 0"/>
         <limit
             lower="-1.83"
@@ -36,9 +36,9 @@
         <parent link="link2"/>
         <child link="link3"/>
-        <origin xyz="0.20 0 0"
-                rpy="0 0 3.1416"/>
-        <axis xyz="0 0 1"/>
+        <origin xyz="0 0.0875 0.200"
+                rpy="0 0 0"/>
+        <axis xyz="0 1 0"/>
         <limit
-            lower="0.0"
+            lower="-2.79"
             upper="2.79"
             effort="100"
@@ -51,7 +51,7 @@
         <parent link="link3"/>
         <child link="link4"/>
-        <origin xyz="0.18 0 0"
-                rpy="-1.5708 0 0"/>
-        <axis xyz="0 0 1"/>
+        <origin xyz="-0.04315 -0.04825 0"
+                rpy="0 0 0"/>
+        <axis xyz="1 0 0"/>
         <limit
             lower="-2.90"
@@ -66,7 +66,7 @@
         <parent link="link4"/>
         <child link="link5"/>
-        <origin xyz="0 0 0.08"
-                rpy="1.5708 0 0"/>
-        <axis xyz="0 0 1"/>
+        <origin xyz="0.22015 0.0435 0"
+                rpy="0 0 0"/>
+        <axis xyz="0 1 0"/>
         <limit
             lower="-2.70"
@@ -81,7 +81,7 @@
         <parent link="link5"/>
         <child link="link6"/>
-        <origin xyz="0 0 0.07"
-                rpy="-1.5708 0 0"/>
-        <axis xyz="0 0 1"/>
+        <origin xyz="0.032324 -0.0435 0"
+                rpy="0 0 0"/>
+        <axis xyz="1 0 0"/>
         <limit
             lower="-3.1416"
@@ -96,5 +96,5 @@
         <parent link="link6"/>
         <child link="tool0"/>
-        <origin xyz="0 0 0.05"
+        <origin xyz="0.022676 0 0"
                 rpy="0 0 0"/>
     </joint>

File: install/robot_description/share/robot_description/urdf/links.xacro (robot description, xacro)
@@ -1,235 +1,61 @@
 <?xml version="1.0"?>
 <robot xmlns:xacro="http://www.ros.org/wiki/xacro">
-    <!-- ===================================================== -->
-    <!-- Base Link -->
-    <!-- ===================================================== -->
-    <link name="base_link">
-        <visual>
-            <origin xyz="0 0 0.05" rpy="0 0 0"/>
-            <geometry>
-                <box size="0.10 0.10 0.10"/>
-            </geometry>
-            <material name="blue"/>
-        </visual>
-        <collision>
-            <origin xyz="0 0 0.05" rpy="0 0 0"/>
-            <geometry>
-                <box size="0.10 0.10 0.10"/>
-            </geometry>
-        </collision>
-        <inertial>
-            <origin xyz="0 0 0.05" rpy="0 0 0"/>
-            <mass value="2.0"/>
-            <inertia
-                ixx="0.005"
-                ixy="0.0"
-                ixz="0.0"
-                iyy="0.005"
-                iyz="0.0"
-                izz="0.005"/>
-        </inertial>
-    </link>
-    <!-- ===================================================== -->
-    <!-- Link 1 : Shoulder Support -->
-    <!-- ===================================================== -->
-    <link name="link1">
-        <visual>
-            <origin xyz="0 0 0.075" rpy="0 0 0"/>
-            <geometry>
-                <box size="0.08 0.08 0.15"/>
-            </geometry>
-            <material name="grey"/>
-        </visual>
-        <collision>
-            <origin xyz="0 0 0.075" rpy="0 0 0"/>
-            <geometry>
-                <box size="0.08 0.08 0.15"/>
-            </geometry>
-        </collision>
-        <inertial>
-            <origin xyz="0 0 0.075" rpy="0 0 0"/>
-            <mass value="1.5"/>
-            <inertia
-                ixx="0.002"
-                ixy="0.0"
-                ixz="0.0"
-                iyy="0.002"
-                iyz="0.0"
-                izz="0.002"/>
-        </inertial>
-    </link>
-    <!-- ===================================================== -->
-    <!-- Link 2 : Upper Arm -->
-    <!-- ===================================================== -->
-    <link name="link2">
-        <visual>
-            <origin xyz="0.10 0 0" rpy="0 0 0"/>
-            <geometry>
-                <box size="0.20 0.05 0.05"/>
-            </geometry>
-            <material name="grey"/>
-        </visual>
-        <collision>
-            <origin xyz="0.10 0 0" rpy="0 0 0"/>
-            <geometry>
-                <box size="0.20 0.05 0.05"/>
-            </geometry>
-        </collision>
-        <inertial>
-            <origin xyz="0.10 0 0" rpy="0 0 0"/>
-            <mass value="1.2"/>
-            <inertia
-                ixx="0.002"
-                ixy="0.0"
-                ixz="0.0"
-                iyy="0.002"
-                iyz="0.0"
-                izz="0.002"/>
-        </inertial>
-    </link>
-    <!-- ===================================================== -->
-    <!-- Link 3 : Forearm -->
-    <!-- ===================================================== -->
-    <link name="link3">
-        <visual>
-            <origin xyz="0.09 0 0" rpy="0 0 0"/>
-            <geometry>
-                <box size="0.18 0.045 0.045"/>
-            </geometry>
-            <material name="grey"/>
-        </visual>
-        <collision>
-            <origin xyz="0.09 0 0" rpy="0 0 0"/>
-            <geometry>
-                <box size="0.18 0.045 0.045"/>
-            </geometry>
-        </collision>
-        <inertial>
-            <origin xyz="0.09 0 0" rpy="0 0 0"/>
-            <mass value="1.0"/>
-            <inertia
-                ixx="0.0015"
-                ixy="0.0"
-                ixz="0.0"
-                iyy="0.0015"
-                iyz="0.0"
-                izz="0.0015"/>
-        </inertial>
-    </link>
-    <!-- ===================================================== -->
-    <!-- Link 4 : Wrist 1 -->
-    <!-- ===================================================== -->
-    <link name="link4">
-        <visual>
-            <origin xyz="0 0 0.04" rpy="0 0 0"/>
-            <geometry>
-                <cylinder radius="0.03" length="0.08"/>
-            </geometry>
-            <material name="grey"/>
-        </visual>
-        <collision>
-            <origin xyz="0 0 0.04" rpy="0 0 0"/>
-            <geometry>
-                <cylinder radius="0.03" length="0.08"/>
-            </geometry>
-        </collision>
-        <inertial>
-            <origin xyz="0 0 0.04" rpy="0 0 0"/>
-            <mass value="0.5"/>
-            <inertia
-                ixx="0.0005"
-                ixy="0.0"
-                ixz="0.0"
-                iyy="0.0005"
-                iyz="0.0"
-                izz="0.0005"/>
-        </inertial>
-    </link>
-    <!-- ===================================================== -->
-    <!-- Link 5 : Wrist 2 -->
-    <!-- ===================================================== -->
-    <link name="link5">
-        <visual>
-            <origin xyz="0 0 0.035" rpy="0 0 0"/>
-            <geometry>
-                <cylinder radius="0.025" length="0.07"/>
-            </geometry>
-            <material name="grey"/>
-        </visual>
-        <collision>
-            <origin xyz="0 0 0.035" rpy="0 0 0"/>
-            <geometry>
-                <cylinder radius="0.025" length="0.07"/>
-            </geometry>
-        </collision>
-        <inertial>
-            <origin xyz="0 0 0.035" rpy="0 0 0"/>
-            <mass value="0.4"/>
-            <inertia
-                ixx="0.0004"
-                ixy="0.0"
-                ixz="0.0"
-                iyy="0.0004"
-                iyz="0.0"
-                izz="0.0004"/>
-        </inertial>
-    </link>
-    <!-- ===================================================== -->
-    <!-- Link 6 : Flange -->
-    <!-- ===================================================== -->
-    <link name="link6">
-        <visual>
-            <origin xyz="0 0 0.025" rpy="0 0 0"/>
-            <geometry>
-                <cylinder radius="0.04" length="0.05"/>
-            </geometry>
-            <material name="grey"/>
-        </visual>
-        <collision>
-            <origin xyz="0 0 0.025" rpy="0 0 0"/>
-            <geometry>
-                <cylinder radius="0.04" length="0.05"/>
-            </geometry>
-        </collision>
-        <inertial>
-            <origin xyz="0 0 0.025" rpy="0 0 0"/>
-            <mass value="0.3"/>
-            <inertia
-                ixx="0.0003"
-                ixy="0.0"
-                ixz="0.0"
-                iyy="0.0003"
-                iyz="0.0"
-                izz="0.0003"/>
-        </inertial>
-    </link>
-    <!-- ===================================================== -->
+    <!-- //Base link -->
+    <xacro:mesh_link
+        name="base_link"
+        mesh="Base_Link.stl"
+        mass="2.0"
+        ixx="0.005"
+        iyy="0.005"
+        izz="0.005"/>
+    <!-- Link 1 -->
+    <xacro:mesh_link
+        name="link1"
+        mesh="Link1.stl"
+        mass="1.5"
+        ixx="0.002"
+        iyy="0.002"
+        izz="0.002"/>
+    <!-- Link 2 -->
+    <xacro:mesh_link
+        name="link2"
+        mesh="Link2.stl"
+        mass="1.2"
+        ixx="0.002"
+        iyy="0.002"
+        izz="0.002"/>
+    <!-- Link 3 -->
+    <xacro:mesh_link
+        name="link3"
+        mesh="Link3.stl"
+        mass="1.0"
+        ixx="0.0015"
+        iyy="0.0015"
+        izz="0.0015"/>
+    <!-- Link 4 -->
+    <xacro:mesh_link
+        name="link4"
+        mesh="Link4.stl"
+        mass="0.5"
+        ixx="0.0005"
+        iyy="0.0005"
+        izz="0.0005"/>
+    <!-- Link 5 -->
+    <xacro:mesh_link
+        name="link5"
+        mesh="Link5.stl"
+        mass="0.4"
+        ixx="0.0004"
+        iyy="0.0004"
+        izz="0.0004"/>
+    <!-- Link 6 -->
+    <xacro:mesh_link
+        name="link6"
+        mesh="Link6.stl"
+        mass="0.3"
+        ixx="0.0003"
+        iyy="0.0003"
+        izz="0.0003"/>
     <!-- Tool Frame -->
-    <!-- ===================================================== -->
-    <link name="tool0">
-        <visual>
-            <origin xyz="0 0 0.02" rpy="0 0 0"/>
-            <geometry>
-                <sphere radius="0.015"/>
-            </geometry>
-            <material name="black"/>
-        </visual>
-        <collision>
-            <origin xyz="0 0 0.02" rpy="0 0 0"/>
-            <geometry>
-                <sphere radius="0.015"/>
-            </geometry>
-        </collision>
-        <inertial>
-            <origin xyz="0 0 0.02" rpy="0 0 0"/>
-            <mass value="0.1"/>
-            <inertia
-                ixx="0.0001"
-                ixy="0.0"
-                ixz="0.0"
-                iyy="0.0001"
-                iyz="0.0"
-                izz="0.0001"/>
-        </inertial>
-    </link>
+    <link name="tool0"/>
 </robot>

File: install/robot_description/share/robot_description/urdf/macros.xacro (robot description, xacro)
@@ -1,3 +1,37 @@
 <?xml version="1.0"?>
 <robot xmlns:xacro="http://www.ros.org/wiki/xacro">
+    <xacro:macro name="mesh_link"
+                 params="
+                    name
+                    mesh
+                    mass
+                    ixx iyy izz
+                    ixy:=0
+                    ixz:=0
+                    iyz:=0
+                    ">
+        <link name="${name}">
+            <visual>
+                <origin xyz="0 0 0" rpy="0 0 0"/>
+                <geometry>
+                    <mesh filename="file:///home/shubham/robot_arm_ws/src/robot_description/meshes/${mesh}"
+                    scale="1 1 1"/>
+                </geometry>
+                <material name="grey"/>
+            </visual>
+            <collision>
+                <origin xyz="0 0 0" rpy="0 0 0"/>
+                <geometry>
+                    <mesh filename="file:///home/shubham/robot_arm_ws/src/robot_description/meshes/${mesh}"
+                        scale="1 1 1"/>
+                </geometry>
+            </collision>
+            <inertial>
+                <origin xyz="0 0 0" rpy="0 0 0"/>
+                <mass value="${mass}"/>
+                <inertia ixx="${ixx}" iyy="${iyy}" izz="${izz}"
+                ixy="${ixy}" ixz="${ixz}" iyz="${iyz}"/>
+            </inertial>
+        </link>
+    </xacro:macro>
 </robot>

File: install/robot_description/share/robot_description/urdf/robot.urdf.xacro (robot description, xacro)
@@ -1,5 +1,5 @@
 <?xml version="1.0"?>
 <robot xmlns:xacro="http://www.ros.org/wiki/xacro"
-       name="robot_arm">
+       name="helene_robot">
     <xacro:include filename="$(find robot_description)/urdf/materials.xacro"/>
     <xacro:include filename="$(find robot_description)/urdf/macros.xacro"/>

File: install/robot_description/share/robot_description/urdf/transmissions.xacro (robot description, xacro)
@@ -1,3 +1,39 @@
 <?xml version="1.0"?>
 <robot xmlns:xacro="http://www.ros.org/wiki/xacro">
+    <!-- ros2_control Configuration -->
+     <ros2_control name="RobotArmSystem" type="system">
+        <hardware>
+            <plugin>gazebo_ros2_control/GazeboSystem</plugin>
+        </hardware>
+        <joint name="joint_1">
+            <command_interface name="position"/>
+            <state_interface name="position"/>
+            <state_interface name="velocity"/>
+        </joint>
+        <joint name="joint_2">
+            <command_interface name="position"/>
+            <state_interface name="position"/>
+            <state_interface name="velocity"/>
+        </joint>
+        <joint name="joint_3">
+            <command_interface name="position"/>
+            <state_interface name="position"/>
+            <state_interface name="velocity"/>
+        </joint>
+        <joint name="joint_4">
+            <command_interface name="position"/>
+            <state_interface name="position"/>
+            <state_interface name="velocity"/>
+        </joint>
+        <joint name="joint_5">
+            <command_interface name="position"/>
+            <state_interface name="position"/>
+            <state_interface name="velocity"/>
+        </joint>
+        <joint name="joint_6">
+            <command_interface name="position"/>
+            <state_interface name="position"/>
+            <state_interface name="velocity"/>
+        </joint>
+    </ros2_control>
 </robot>
