Commit message: Still Stuck in 1.88 million trianglesin a single robotic arm

File: install/robot_description/share/robot_description/urdf/macros.xacro (robot description, xacro)
@@ -15,6 +15,8 @@
                 <origin xyz="0 0 0" rpy="0 0 0"/>
                 <geometry>
+                    <!-- Debugging -->
                     <mesh filename="file:///home/shubham/robot_arm_ws/src/robot_description/meshes/${mesh}"
                     scale="1 1 1"/>
+                    <!-- <box size="0.2 0.2 0.2"/> -->
                 </geometry>
                 <material name="grey"/>
